Commit message: mapping

File: catkin_ws/src/device_description/urdf/device.urdf (robot description, URDF)
Before this commit: robot duckiefloat, 3 links, 2 joints
Joints:
- joint imu: origin xyz=-0.04 0.1 0 rpy=0 0 0 -> xyz=0.1 0.04 0 rpy=0 0 0
- joint velodyne: origin xyz=0 0 0.1 rpy=0 0 0 -> xyz=0 0 0.25 rpy=0 0 0
